File: pond_filter_schematic/pond_filter_schematic.kicad_sch (KiCad schematic)
At the start: 8 parts, among them J1 Analog, J2 Digital

Commit message: updated resistor value
Parts:
- R1: value 2.2k -> 20k
Changed lines of the file:
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@@
 			)
 		)
-		(property "Value" "2.2k"
+		(property "Value" "20k"
 			(at 123.19 80.0099 0)
 			(show_name no)
